File: src/retro-usb-interface/hw/retro-usb-interface/retro-usb-interface.kicad_sch (KiCad schematic)
At the start: 13 parts, among them J1 Conn_02x05_Odd_Even, J2 Conn_01x04_Pin, J3 Conn_01x03_Pin, J4 Conn_01x05_Pin, Q1 BSS138, U1 MAX3232, U2 Pico

Commit message: retro-usb-interface: restore functionality
This re-enabled mouses support and isolate keyboard functionality (which
is not finished but good enough to keep)

While here, update the schematics.
Parts:
- added D1: LED, symbol Device:LED
- added Q2: BSS138, Package_TO_SOT_SMD:SOT-23, symbol Transistor_FET:BSS138
- added R3, R4: 10k, symbol Device:R
- added R5: R, symbol Device:R
Connections:
- net LV is gone; now on net +3.3V: Q1.1 (G), R1.1
- net LV1 is gone; now on net KBD_CLK_3V3: Q1.2 (S)
- net +3.3V: now also Q2.1 (G), R3.1
- net GND: now also R5.2
- net HV: no longer R2.1
- net HV1: no longer Q1.3 (D)
- net KBD_CLK: now also Q1.3 (D), R2.2
- net KBD_DATA: now also Q2.3 (D), R4.2
- net KBD_VCC: now also R2.1, R4.1
- net KBD_CLK_3V3: now reaches R1.2
- net KBD_CLK_3V3: now also U2.14 (GPIO10), U2.16 (GPIO12)
- net KBD_DATA_3V3: now reaches U2.15 (GPIO11)
- net KBD_DATA_3V3: now also U2.17 (GPIO13), Q2.2 (S)
- net DEBUG_LED1: now reaches U2.20 (GPIO15)
- net DEBUG_LED1: now also D1.2 (A)
- net DEBUG_LED2: now reaches U2.21 (GPIO16)
- net DEBUG_LED3: now reaches U2.22 (GPIO17)
- net GPIO3 renamed MS_DTR
- net GPIO4 renamed MS_TXD
- net GPIO5 renamed MS_RXD
- new net: D1.1 (K), R5.1
- no-connect marks 40 -> 33
Other:
- moved on the sheet: Q1, R1
